File: Devboard.kicad_pcb (KiCad board)
At the start: 2 copper layers, 76 x 48.6 mm, 36 parts, among them J1 Power, J10 terminal, J2 Left, J3 ARM-JTAG, J4 Right, J5 JTAG, J6 Screw_Terminal_01x02, J7 Jack-DC, J8 Power, J9 DNP, Q1 IRF7101, SW1 RESET, U1 TRADFRI, U2 AMS1117-3.3

Commit message: enhancements to pcb, this will be possible rev B
Parts:
- moved SW1 39.2 mm to (178.3, 133.6), turned to 90 degrees
- moved JP4 9.12 mm to (189.1, 126.5)
- moved J4 5.02 mm to (180.3, 97.5)
- moved U1 4.82 mm to (165.6, 91.7)
- moved C2 4.32 mm to (151.4, 115.1), turned to 180 degrees
Routing:
- net GND: track 60.4 -> 43.3 mm, vias 61 -> 118
- net /RESETn: track 94.7 -> 79.7 mm
- net /SWCLK: track 53.1 -> 42.9 mm, vias 0 -> 1
- net /SWO: track 38.4 -> 44.7 mm
- net +3V3: track 105.8 -> 111.6 mm
- net Net-(J2-Pad3): track 25.3 -> 22.9 mm
- net Net-(J10-Pad4): track 26.3 -> 24.0 mm
- net Net-(J2-Pad1): track 10.1 -> 8.04 mm
- net Net-(J4-Pad2): track 9.57 -> 11.2 mm
- net Net-(J2-Pad2): track 9.85 -> 8.35 mm
- net Net-(J4-Pad6): track 10.7 -> 11.8 mm
- net /SWDIO: track 48.0 -> 49.0 mm
- net Net-(J10-Pad2): track 23.0 -> 22.3 mm
- net Net-(J2-Pad4): track 25.5 -> 24.7 mm
Other:
- board text added: "1"
- board text added: "IRF7101"
- board text added: "rev. B"
